Commit message: fixed pendulum swing

File: DigitalControl/dynamic_tests/test.urdf (robot description, URDF)
Before this commit: robot bender, 4 links, 3 joints
Links:
- link link_1: mass 6 -> 1
- link link_eef: mass 100 -> 1

Commit message: pid-regulator for 1 joint

File: DigitalControl/dynamic_tests/test.urdf (robot description, URDF)
Before this commit: robot bender, 4 links, 3 joints
Joints:
- joint joint_1: origin xyz=0.0 0 -0.1 rpy=0 1.57 0 -> xyz=0.0 0 -0.1 rpy=0 0 0
