Commit message: better appearance of the pendulum

File: DigitalControl/dynamic_tests/simple.urdf (robot description, URDF)
Before this commit: robot bender, 4 links, 3 joints
Links:
- link base: geometry visual sphere radius=0.1
- link link_1: geometry visual cylinder length=0.8 radius=0.01
- link link_eef: geometry visual sphere radius=0.05
Joints:
- joint joint_1: origin xyz=0.0 0 -0.3 rpy=0 3.14159265358979323846 0 -> xyz=0.0 0 0 rpy=0 3.14159265358979323846 0

Commit message: ideal pid + camera basics

File: DigitalControl/dynamic_tests/simple.urdf (robot description, URDF)
Before this commit: robot bender, 4 links, 3 joints
Links:
- added link code; visual mesh filename=meshes2/files/alternative_white.stl scale=0.00251
- added link code_bg; visual box size=0.1 0.1 0.1
Joints:
- added joint box_bg: type fixed, parent code, child code_bg
- added joint box_w: type fixed, parent world, child code, origin xyz=1 0 0 rpy=0 0 0

Commit message: working aruco-detector

File: DigitalControl/dynamic_tests/simple.urdf (robot description, URDF)
Before this commit: robot bender, 6 links, 5 joints
Links:
- link code: geometry visual mesh filename=meshes2/files/arucocube_black.stl scale=0.00251
