Commit message: working aruco pose estimation

File: DigitalControl/dynamic_tests/marker.urdf (robot description, URDF)
Before this commit: robot marker, 3 links, 2 joints
Links:
- link marker: geometry visual mesh filename=meshes2/files/arucocube_black.stl scale=0.0051
- link marker_background: geometry visual box size=0.22 0.22 0.2
Joints:
- joint world_to_marker: origin xyz=0 0 0 rpy=0 0 0 -> xyz=0.1 0.1 0 rpy=0 0 0
