Commit message: added one more link and joint

File: DigitalControl/robot.urdf (robot description, URDF)
Before this commit: robot bender, 2 links, 1 joints
Links:
- added link link_1; visual cylinder length=0.4 radius=0.1
- link base: geometry visual cylinder length=0.2 radius=0.3
Joints:
- added joint base_to_link_1: type revolute, parent base, child link_1, origin xyz=0 0 0.3 rpy=0 0 0, limit lower=-3.15 upper=3.15
- joint world_to_base: origin xyz=0 0 0 rpy=0 0 0 -> xyz=0 0 0.1 rpy=0 0 0

Commit message: another link and joint

File: DigitalControl/robot.urdf (robot description, URDF)
Before this commit: robot bender, 3 links, 2 joints
Links:
- added link link_2; visual cylinder length=0.8 radius=0.05
Joints:
- removed joint base_to_link_1
- added joint joint_1: type revolute, parent base, child link_1, origin xyz=0.2 0 0.2 rpy=0 1.57 0, axis 0 0 1, limit lower=-3.15 upper=3.15
- added joint joint_2: type revolute, parent link_1, child link_2, origin xyz=-0.4 0 0.2 rpy=0 -1.57 0, axis 0 1 0, limit lower=-3.15 upper=3.15

Commit message: assuming direct control...

File: DigitalControl/robot.urdf (robot description, URDF)
Before this commit: robot bender, 4 links, 3 joints
Joints:
- joint joint_1: axis 0 0 1 -> 1 0 0; origin xyz=0.2 0 0.2 rpy=0 1.57 0 -> xyz=0.0 0 0.2 rpy=0 1.57 0
- joint joint_2: origin xyz=-0.4 0 0.2 rpy=0 -1.57 0 -> xyz=0 0 0.4 rpy=0 -1.57 0

Commit message: added fk service

File: DigitalControl/robot.urdf (robot description, URDF)
Before this commit: robot bender, 4 links, 3 joints
Links:
- added link link_eef; visual cylinder length=0.1 radius=0.05
Joints:
- added joint joint_eef: type fixed, parent link_2, child link_eef, origin xyz=0 0 0.8 rpy=0 0 0

Commit message: full 6DoF robot

File: DigitalControl/robot.urdf (robot description, URDF)
Before this commit: robot bender, 5 links, 4 joints
Links:
- added link link_3
- added link link_4; visual cylinder length=0.4 radius=0.05
- added link link_5; visual cylinder length=0.2 radius=0.05
- added link link_6
- link link_eef: geometry visual box size=0.1 0.1 0.1
Joints:
- added joint joint_3: type revolute, parent link_2, child link_3, origin xyz=0 0 0.8 rpy=0 0 0, axis 0 1 0, limit lower=-3.15 upper=3.15
- added joint joint_4: type revolute, parent link_3, child link_4, origin xyz=0 0 0 rpy=0 0 0, axis 0 0 1, limit lower=-3.15 upper=3.15
- added joint joint_5: type revolute, parent link_4, child link_5, origin xyz=0 0 0.4 rpy=0 0 0, axis 0 1 0, limit lower=-3.15 upper=3.15
- added joint joint_6: type revolute, parent link_5, child link_6, origin xyz=0 0 0 rpy=0 0 0, axis 0 0 1, limit lower=-3.15 upper=3.15
- joint joint_eef: origin xyz=0 0 0.8 rpy=0 0 0 -> xyz=0 0 0.2 rpy=0 0 0; parent link_2 -> link_6

Commit message: added camera following to robot

File: DigitalControl/robot.urdf (robot description, URDF)
Before this commit: robot bender, 9 links, 8 joints
Links:
- added link marker; visual mesh filename=dynamic_tests/meshes2/files/arucocube_black.stl scale=0.0051
- added link marker_background; visual box size=0.22 0.22 0.2
- added link marker_base
- link link_2: mass None -> 5
- link link_eef: mass None -> 0
Joints:
- added joint base_to_marker: type fixed, parent marker_base, child marker, origin xyz=0 0 0 rpy=0 0 0
- added joint marker_to_bg: type fixed, parent marker, child marker_background
- added joint world_to_marker_base: type prismatic, parent world, child marker_base, origin xyz=3 0 0.5 rpy=0 -1.5708 0, limit lower=-1 upper=1 velocity=1
